File: Nanostripes_Connector/Nanostripes_Connector.kicad_pcb (KiCad board)
At the start: 2 copper layers, 32 x 37 mm, 20 parts, among them J1 Input_E1, J2 Input_E2, J3 Input_E3, J4 Input_E4, J5 Input_E5, J6 Input_E6, J8 Conn_01x04_Pin, U1 78L03, U2 ATSAMD11D14A-M

Commit message: finished and panelized
Parts:
- C1, C2, D1, R1, R2, R3, R4, R5, R6, R7, U1: moved to B.Cu
- moved U1 8.00 mm to (65.8, 61.5), turned to 180 degrees
- moved C1 7.52 mm to (65.8, 64.2), turned to 180 degrees
- moved D1 6.67 mm to (71.2, 60.5), turned to -90 degrees
- moved C3 6.01 mm to (62.2, 50.8), turned to 0 degrees
- moved C2 5.43 mm to (69.0, 61.5), turned to -90 degrees
- moved U2 4.65 mm to (64.2, 54.9)
- moved J8 1.02 mm to (59.0, 55.5)
- moved R1 0.90 mm to (69.2, 64.2), turned to 180 degrees
- moved R4 0.25 mm to (77.5, 50.2)
Routing:
- net GND: track 11.1 -> 3.43 mm
- net Net-(U2-PA14): track 19.9 -> 13.4 mm, vias 1 -> 2
- net Net-(U2-PA24): track 18.3 -> 24.2 mm, vias 3 -> 2
- net Net-(U2-PA04): track 16.1 -> 12.3 mm, vias 1 -> 0
- net Net-(U2-PA16): track 14.3 -> 17.2 mm, vias 1 -> 2
- net Net-(U2-PA10): track 25.9 -> 23.4 mm, vias 3 -> 4
- net +42V: track 0.00 -> 2.50 mm, vias 0 -> 2
- net +3.3V: track 23.1 -> 25.1 mm, vias 1 -> 3
- net SWCLK: track 4.81 -> 6.59 mm
- net Net-(U1-IN): track 4.57 -> 3.52 mm
- net Net-(U2-PA08/XIN): track 14.1 -> 13.0 mm, vias 5 -> 2
- net SWDIO: track 5.04 -> 4.27 mm
- net /Controller/E2: track 3.61 -> 4.34 mm
- net /Controller/E5: track 3.71 -> 4.39 mm
Other:
- board text added: "E1"
- board text added: "E2"
