File: Nanostripes_Connector/controller.kicad_sch (KiCad schematic)
At the start: 9 parts, among them J8 Conn_01x04_Pin, U2 ATSAMD11D14A-M

Commit message: updated component values
Parts:
- C3: value 100n -> 100nF
Changed lines of the file:
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@@
 			)
 		)
-		(property "Value" "100n"
+		(property "Value" "100nF"
 			(at 29.21 31.7499 0)
 			(effects
