File: Nanostripes_LED_Modul/Nanostripes_LED_Modul.kicad_pcb (KiCad board)
At the start: 2 copper layers, 275 x 15 mm, 95 parts, among them J1 Input_E1, J2 Input_E1_Test, J3 Input_E2, J4 Input_E2_Test, J5 Conn_01x02_Pin, J6 Conn_01x02_Pin, J7 Conn_01x02_Pin, J8 Conn_01x02_Pin, Q1 BC 846B, Q2 BC 846B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

Commit message: finished and panelized
Routing:
- net GND: track 41.3 -> 43.1 mm
Other:
- board text added: "E1"
Changed lines of the file:
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@@
 		(sheetname "Controller")
 		(sheetfile "controller.kicad_sch")
-		(attr through_hole)
+		(attr through_hole exclude_from_pos_files exclude_from_bom)
 		(fp_line
 			(start -1.33 3.87)
@@
 		(sheetname "Stammblatt")
 		(sheetfile "Nanostripes_LED_Modul.kicad_sch")
-		(attr through_hole)
+		(attr through_hole exclude_from_pos_files exclude_from_bom)
 		(fp_line
 			(start -1.33 -1.33)
@@
 		(sheetname "Stammblatt")
 		(sheetfile "Nanostripes_LED_Modul.kicad_sch")
-		(attr through_hole)
+		(attr through_hole exclude_from_pos_files exclude_from_bom)
 		(fp_line
 			(start 1.33 1.27)
@@
 		(sheetname "Controller")
 		(sheetfile "controller.kicad_sch")
-		(attr through_hole)
+		(attr through_hole exclude_from_pos_files exclude_from_bom)
 		(fp_line
 			(start -1.33 -1.33)
@@
 		(tags "Through hole pin header THT 1x02 2.54mm single row")
 		(property "Reference" "J6"
-			(at 0 -2.33 -90)
+			(at 0 -2.33 90)
 			(layer "F.SilkS")
 			(effects
@@
 		)
 		(property "Value" "Conn_01x02_Pin"
-			(at 0 4.87 -90)
+			(at 0 4.87 90)
 			(layer "F.Fab")
 			(effects
@@
 		(sheetname "Controller")
 		(sheetfile "controller.kicad_sch")
-		(attr through_hole)
+		(attr through_hole exclude_from_pos_files exclude_from_bom)
 		(fp_line
 			(start -1.33 3.87)
@@
 		(sheetname "Controller")
 		(sheetfile "controller.kicad_sch")
-		(attr through_hole)
+		(attr through_hole exclude_from_pos_files exclude_from_bom)
 		(fp_line
 			(start -1.33 -1.33)
@@
 		(sheetname "Stammblatt")
 		(sheetfile "Nanostripes_LED_Modul.kicad_sch")
-		(attr through_hole)
+		(attr through_hole exclude_from_pos_files exclude_from_bom)
 		(fp_line
 			(start -1.33 -1.33)
@@
 		(sheetname "Stammblatt")
 		(sheetfile "Nanostripes_LED_Modul.kicad_sch")
-		(attr through_hole)
+		(attr through_hole exclude_from_pos_files exclude_from_bom)
 		(fp_line
 			(start -1.33 -1.33)
@@
 		(layer "User.1")
 	)
+	(gr_text "E1"
+		(at 53 78 0)
+		(layer "F.SilkS")
+		(effects
+			(font
+				(size 1 1)
+				(thickness 0.15)
+			)
+			(justify left bottom)
+		)
+	)
 	(gr_text "SWDIO\nSWCLK"
 		(at 143.75 84.75 90)
@@
 	)
 	(segment
-		(start 137.5 79.2)
+		(start 252.7 86.25)
+		(end 253.25 85.7)
+		(width 0.2)
+		(layer "F.Cu")
+		(net 1)
+	)
+	(segment
+		(start 138.2 79.55)
 		(end 138.2 78.5)
 		(width 0.2)
@@
 	)
 	(segment
-		(start 252.7 86.25)
-		(end 253.25 85.7)
+		(start 62.25 82.95)
+		(end 61.3 82)
 		(width 0.2)
 		(layer "F.Cu")
@@
 	)
 	(segment
-		(start 137.5 81.0625)
-		(end 137.5 79.2)
+		(start 61.3 82)
+		(end 60.75 82)
+		(width 0.2)
+		(layer "F.Cu")
+		(net 1)
+	)
+	(segment
+		(start 137.5 80.25)
+		(end 138.2 79.55)
 		(width 0.2)
 		(layer "F.Cu")
@@
 	)
 	(segment
+		(start 137.5 81.0625)
+		(end 137.5 80.25)
+		(width 0.2)
+		(layer "F.Cu")
+		(net 1)
+	)
+	(segment
 		(start 250 86)
 		(end 250 84.9375)
@@
 		(polygon
 			(pts
-				(xy 40 70) (xy 330 70) (xy 330 95) (xy 40 95)
+				(xy 48 75) (xy 323 75) (xy 323 90) (xy 48 90)
 			)
 		)
@@
 		(polygon
 			(pts
-				(xy 40 70) (xy 330 70) (xy 330 95) (xy 40 95)
+				(xy 48 75) (xy 323 75) (xy 323 90) (xy 48 90)
 			)
 		)

Commit message: updated component values
Parts:
- R10, R11, R12, R18, R19, R20, R21, R9: value 120 -> 1k
Changed lines of the file:
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@@
 			)
 		)
-		(property "Value" "120"
+		(property "Value" "1k"
 			(at 0 1.65 0)
 			(layer "F.Fab")
@@
 			)
 		)
-		(property "Value" "120"
+		(property "Value" "1k"
 			(at 0 1.65 0)
 			(layer "F.Fab")
@@
 			)
 		)
-		(property "Value" "120"
+		(property "Value" "1k"
 			(at 0 1.65 0)
 			(layer "F.Fab")
@@
 		(sheetname "Controller")
 		(sheetfile "controller.kicad_sch")
-		(attr through_hole exclude_from_pos_files exclude_from_bom)
+		(attr through_hole exclude_from_pos_files)
 		(fp_line
 			(start -1.33 3.87)
@@
 		(sheetname "Stammblatt")
 		(sheetfile "Nanostripes_LED_Modul.kicad_sch")
-		(attr through_hole exclude_from_pos_files exclude_from_bom)
+		(attr through_hole exclude_from_pos_files)
 		(fp_line
 			(start -1.33 -1.33)
@@
 			)
 		)
-		(property "Value" "120"
+		(property "Value" "1k"
 			(at 0 1.65 0)
 			(layer "F.Fab")
@@
 		(sheetname "Stammblatt")
 		(sheetfile "Nanostripes_LED_Modul.kicad_sch")
-		(attr through_hole exclude_from_pos_files exclude_from_bom)
+		(attr through_hole exclude_from_pos_files)
 		(fp_line
 			(start 1.33 1.27)
@@
 		(sheetname "Controller")
 		(sheetfile "controller.kicad_sch")
-		(attr through_hole exclude_from_pos_files exclude_from_bom)
+		(attr through_hole exclude_from_pos_files)
 		(fp_line
 			(start -1.33 -1.33)
@@
 			)
 		)
-		(property "Value" "120"
+		(property "Value" "1k"
 			(at 0 1.65 0)
 			(layer "F.Fab")
@@
 		(sheetname "Controller")
 		(sheetfile "controller.kicad_sch")
-		(attr through_hole exclude_from_pos_files exclude_from_bom)
+		(attr through_hole exclude_from_pos_files)
 		(fp_line
 			(start -1.33 3.87)
@@
 			)
 		)
-		(property "Value" "120"
+		(property "Value" "1k"
 			(at 0 1.65 0)
 			(layer "F.Fab")
@@
 		(sheetname "Controller")
 		(sheetfile "controller.kicad_sch")
-		(attr through_hole exclude_from_pos_files exclude_from_bom)
+		(attr through_hole exclude_from_pos_files)
 		(fp_line
 			(start -1.33 -1.33)
@@
 			)
 		)
-		(property "Value" "120"
+		(property "Value" "1k"
 			(at 0 1.65 0)
 			(layer "F.Fab")
@@
 		(sheetname "Stammblatt")
 		(sheetfile "Nanostripes_LED_Modul.kicad_sch")
-		(attr through_hole exclude_from_pos_files exclude_from_bom)
+		(attr through_hole exclude_from_pos_files)
 		(fp_line
 			(start -1.33 -1.33)
@@
 		(sheetname "Stammblatt")
 		(sheetfile "Nanostripes_LED_Modul.kicad_sch")
-		(attr through_hole exclude_from_pos_files exclude_from_bom)
+		(attr through_hole exclude_from_pos_files)
 		(fp_line
 			(start -1.33 -1.33)
@@
 			)
 		)
-		(property "Value" "120"
+		(property "Value" "1k"
 			(at 0 1.65 0)
 			(layer "F.Fab")
