File: Nanostripes_LED_Modul/controller.kicad_sch (KiCad schematic)
At the start: 12 parts, among them J5 Conn_01x02_Pin, J6 Conn_01x02_Pin, J7 Conn_01x02_Pin, J8 Conn_01x02_Pin, U2 ATSAMD11D14A-M, U3 ATSAMD11D14A-M

Commit message: updated component values
Parts:
- C3, C4: value 100n -> 100nF
Changed lines of the file:
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@@
 			)
 		)
-		(property "Value" "100n"
+		(property "Value" "100nF"
 			(at 29.21 31.7499 0)
 			(effects
@@
 			)
 		)
-		(property "Value" "100n"
+		(property "Value" "100nF"
 			(at 29.21 102.8699 0)
 			(effects
